File: UART Card/UART Card.kicad_pcb (KiCad board)
At the start: 2 copper layers, 100 x 100 mm, 30 parts, among them J1 Conn_02x20_Odd_Even, J2 DB9_ Male, U1 74LS00, U2 MAX232, U3 CDP1854AE, U4 74LS393, U5 74LS157, U6 MCP2221AxP, X1 CXO_DIP8

Commit message: Finalised board layout
Parts:
- moved C10 2.49 mm to (135.1, 101.7), turned to 180 degrees
- moved C6 0.36 mm to (118.0, 70.9)
Routing:
- net GND: track 409.2 -> 340.5 mm
- net VCC: track 198.5 -> 171.3 mm
- net High: track 142.7 -> 161.8 mm
- net Net-(U2-Pad9): track 53.3 -> 35.9 mm
- net ~CLEAR: track 93.3 -> 105.1 mm
- net Net-(JP4-Pad2): track 75.0 -> 85.5 mm
- net ~N3: track 56.2 -> 47.2 mm, vias 0 -> 2
- net /RX: track 27.2 -> 35.8 mm
- net Net-(JP2-Pad1): track 80.9 -> 72.8 mm
- net Net-(U2-Pad11): track 74.3 -> 66.3 mm, vias 0 -> 1
- net Net-(U3-Pad39): track 71.0 -> 78.8 mm, vias 1 -> 0
- net Net-(JP1-Pad10): track 32.7 -> 25.2 mm
- net TPB: track 48.9 -> 56.3 mm
- net /CTS: track 42.3 -> 48.4 mm
- net /TX: track 23.6 -> 29.7 mm
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Other:
- board text added: "JP1 - Baud Rate Selection JP2 - USB - On = RS232 via USB, Off = via DB-9 JP3 - Interrupt - Enables Interrupts JP4 - EF4 - Allow EF4 to detect USB or RS232 connection Q - 1854 Register Select (RSEL) N3 - 1854 Register Read/Write"
- board text removed: "1854 UART Card Rev.1.0"
- board text removed: "JP1 - Baud Rate Selection JP2 - USB - On = USB connection, Off = RS232 JP3 - Interrupt - Enables Interrupts JP4 - EF4 - Allow EF4 to detect USB or RS232 connection Q - Register Select (RSEL)"
