File: UART Card/UART Card.sch (KiCad schematic (older format))
At the start: 29 parts, among them J1 Conn_02x20_Odd_Even, J2 DB9_ Male, U1 74LS00, U2 MAX232, U3 CDP1854AE, U4 74LS393, U5 74LS157, U6 MCP2221AxP, X1 CXO_DIP8

Commit message: Finalised board layout
Connections:
- no-connect marks 18 -> 20
Changed lines of the file:
@@
 	1    0    0    -1
 $EndComp
+NoConn ~ 8450 2200
+NoConn ~ 8450 2100
 Wire Wire Line
 	4450 5450 5450 5450
 Wire Bus Line
+	2350 4450 2350 7450
+Wire Bus Line
 	5200 4750 5200 7450
-Wire Bus Line
-	2350 4450 2350 7450
 $EndSCHEMATC
